Commit message: complete assignment 01: add rgb camera

File: src/arduinobot_description/urdf/arduinobot.urdf.xacro (robot description, xacro)
@@ -114,3 +114,17 @@
 		<limit lower="0.0" upper="${PI/2}" effort="${effort}" velocity="${velocity}"></limit>
 	</joint>
+	<link name="rgb_camera">
+		<visual>
+			<origin xyz="-0.08 0.125 0.125" rpy="-${PI/2} 0 -${PI/2}"></origin>
+			<geometry>
+				<mesh filename="package://arduinobot_description/meshes/pi_camera.STL"
+					scale="0.01 0.01 0.01"></mesh>
+			</geometry>
+		</visual>
+	</link>
+	<joint name="joint_6" type="fixed">
+		<parent link="base_link" />
+		<child link="rgb_camera" />
+		<origin rpy="0 -0.5 1.57" xyz="0 0.45 0.2" />
+	</joint>
 </robot>

Commit message: complete section 05. Control

File: src/arduinobot_description/urdf/arduinobot.urdf.xacro (robot description, xacro)
@@ -1,9 +1,29 @@
 <?xml version="1.0"?>
 <robot xmlns:xacro="http://www.ros.org/wiki/xacro" name="arduinobot">
+	<xacro:include filename="$(find arduinobot_description)/urdf/arduinobot_gazebo.xacro" />
+	<xacro:include filename="$(find arduinobot_description)/urdf/arduinobot_ros2_control.xacro" />
 	<xacro:property name="PI" value="3.14159" />
 	<xacro:property name="effort" value="30.0" />
 	<xacro:property name="velocity" value="10.0" />
+	<xacro:macro name="default_inertial" params="mass">
+		<inertial>
+			<mass value="${mass}"></mass>
+			<inertia ixx="1.0" ixy="0.0" ixz="0.0"
+				iyy="1.0" iyz="0.0"
+				izz="1.0"></inertia>
+		</inertial>
+	</xacro:macro>
+	<xacro:macro name="default_transmission" params="number">
+		<transmission name="transmission_${number}">
+			<plugin>transmission_interface/SimpleTransmission</plugin>
+			<actuator name="motor_${number}" role="actuator1" />
+			<joint name="joint_${number}" role="joint1">
+				<mechanical_reduction>1.0</mechanical_reduction>
+			</joint>
+		</transmission>
+	</xacro:macro>
 	<link name="world" />
 	<link name="base_link">
+		<xacro:default_inertial mass="1.0" />
 		<visual>
 			<origin rpy="0 0 0" xyz="-0.5 -0.5 0" />
@@ -13,4 +33,11 @@
 			</geometry>
 		</visual>
+		<collision>
+			<origin rpy="0 0 0" xyz="-0.5 -0.5 0" />
+			<geometry>
+				<mesh filename="package://arduinobot_description/meshes/basement.STL"
+					scale="0.01 0.01 0.01" />
+			</geometry>
+		</collision>
 	</link>
 	<joint name="virtual_joint" type="fixed">
@@ -20,4 +47,5 @@
 	</joint>
 	<link name="base_plate">
+		<xacro:default_inertial mass="0.1" />
 		<visual>
 			<origin rpy="0 0 0" xyz="-0.39 -0.39 -0.56"></origin>
@@ -27,4 +55,11 @@
 			</geometry>
 		</visual>
+		<collision>
+			<origin rpy="0 0 0" xyz="-0.39 -0.39 -0.56"></origin>
+			<geometry>
+				<mesh filename="package://arduinobot_description/meshes/base_plate.STL"
+					scale="0.01 0.01 0.01"></mesh>
+			</geometry>
+		</collision>
 	</link>
 	<joint name="joint_1" type="revolute">
@@ -36,4 +71,5 @@
 	</joint>
 	<link name="forward_drive_arm">
+		<xacro:default_inertial mass="0.1" />
 		<visual>
 			<origin rpy="0 -${PI/2} ${PI/2}" xyz="0.19 0.06 -0.08"></origin>
@@ -43,4 +79,11 @@
 			</geometry>
 		</visual>
+		<collision>
+			<origin rpy="0 -${PI/2} ${PI/2}" xyz="0.19 0.06 -0.08"></origin>
+			<geometry>
+				<mesh filename="package://arduinobot_description/meshes/forward_drive_arm.STL"
+					scale="0.01 0.01 0.01"></mesh>
+			</geometry>
+		</collision>
 	</link>
 	<joint name="joint_2" type="revolute">
@@ -52,4 +95,5 @@
 	</joint>
 	<link name="horizontal_arm">
+		<xacro:default_inertial mass="0.1" />
 		<visual>
 			<origin rpy="${PI/2} 0 ${PI/2}" xyz="-0.03 -0.4 -0.06"></origin>
@@ -59,4 +103,11 @@
 			</geometry>
 		</visual>
+		<collision>
+			<origin rpy="${PI/2} 0 ${PI/2}" xyz="-0.03 -0.4 -0.06"></origin>
+			<geometry>
+				<mesh filename="package://arduinobot_description/meshes/horizontal_arm.STL"
+					scale="0.01 0.01 0.01"></mesh>
+			</geometry>
+		</collision>
 	</link>
 	<joint name="joint_3" type="revolute">
@@ -68,4 +119,5 @@
 	</joint>
 	<link name="claw_support">
+		<xacro:default_inertial mass="0.05" />
 		<visual>
 			<origin rpy="0 0 ${PI/2}" xyz="0 -0.05 -0.15"></origin>
@@ -75,4 +127,11 @@
 			</geometry>
 		</visual>
+		<collision>
+			<origin rpy="0 0 ${PI/2}" xyz="0 -0.05 -0.15"></origin>
+			<geometry>
+				<mesh filename="package://arduinobot_description/meshes/claw_support.STL"
+					scale="0.01 0.01 0.01"></mesh>
+			</geometry>
+		</collision>
 	</link>
 	<joint name="horizontal_arm_to_claw_support" type="fixed">
@@ -82,4 +141,5 @@
 	</joint>
 	<link name="gripper_right">
+		<xacro:default_inertial mass="0.01" />
 		<visual>
 			<origin xyz="-0.1 0.5 -0.1" rpy="0 0 -${PI/2}"></origin>
@@ -89,6 +149,14 @@
 			</geometry>
 		</visual>
+		<collision>
+			<origin xyz="-0.1 0.5 -0.1" rpy="0 0 -${PI/2}"></origin>
+			<geometry>
+				<mesh filename="package://arduinobot_description/meshes/right_finger.STL"
+					scale="0.01 0.01 0.01"></mesh>
+			</geometry>
+		</collision>
 	</link>
 	<link name="gripper_left">
+		<xacro:default_inertial mass="0.01" />
 		<visual>
 			<origin xyz="-0.04 0.5 -0.1" rpy="0 0 -${PI/2}"></origin>
@@ -98,4 +166,11 @@
 			</geometry>
 		</visual>
+		<collision>
+			<origin xyz="-0.04 0.5 -0.1" rpy="0 0 -${PI/2}"></origin>
+			<geometry>
+				<mesh filename="package://arduinobot_description/meshes/left_finger.STL"
+					scale="0.01 0.01 0.01"></mesh>
+			</geometry>
+		</collision>
 	</link>
 	<joint name="joint_4" type="revolute">
@@ -115,4 +190,5 @@
 	</joint>
 	<link name="rgb_camera">
+		<xacro:default_inertial mass="0.001" />
 		<visual>
 			<origin xyz="-0.08 0.125 0.125" rpy="-${PI/2} 0 -${PI/2}"></origin>
@@ -122,4 +198,11 @@
 			</geometry>
 		</visual>
+		<collision>
+			<origin xyz="-0.08 0.125 0.125" rpy="-${PI/2} 0 -${PI/2}"></origin>
+			<geometry>
+				<mesh filename="package://arduinobot_description/meshes/pi_camera.STL"
+					scale="0.01 0.01 0.01"></mesh>
+			</geometry>
+		</collision>
 	</link>
 	<joint name="joint_6" type="fixed">
@@ -128,3 +211,7 @@
 		<origin rpy="0 -0.5 1.57" xyz="0 0.45 0.2" />
 	</joint>
+	<xacro:default_transmission number="1"/>
+	<xacro:default_transmission number="2"/>
+	<xacro:default_transmission number="3"/>
+	<xacro:default_transmission number="4"/>
 </robot>

Commit message: please continuing at sec.4 lesson 33

File: src/arduinobot_description/urdf/arduinobot.urdf.xacro (robot description, xacro)
@@ -1,6 +1,20 @@
 <?xml version="1.0"?>
+<!-- We are using the xacro format, not plain urdf => we need to indicate where the definition of this format is located  -->
 <robot xmlns:xacro="http://www.ros.org/wiki/xacro" name="arduinobot">
 	<xacro:include filename="$(find arduinobot_description)/urdf/arduinobot_gazebo.xacro" />
 	<xacro:include filename="$(find arduinobot_description)/urdf/arduinobot_ros2_control.xacro" />
+	<!-- Useful XACRO Variables (Properties) -->
+	<!--
+		Since we are going to use the same actuators, so the same motors for all the
+		all movable joints of our robotic arm, basically their mechanical and
+		kinematic limits will be the same. So that we can create some properties
+		to make use of the reusability.
+	-->
+	<!--
+		An actuator is a component of a machine that produces force, torque, or
+		displacement, usually in a controlled way, when an electrical, pneumatic
+		or hydraulic input is supplied to it in a system (called an
+		actuating system).
+	-->
 	<xacro:property name="PI" value="3.14159" />
 	<xacro:property name="effort" value="30.0" />
@@ -23,10 +37,18 @@
 		</transmission>
 	</xacro:macro>
+	<!-- ************ LINK ************  -->
+	<!-- This link serves to anchor the manipulator to the world reference frame -->
 	<link name="world" />
 	<link name="base_link">
 		<xacro:default_inertial mass="1.0" />
-		<visual>
-			<origin rpy="0 0 0" xyz="-0.5 -0.5 0" />
-			<geometry>
+		<!-- Visualize by the visual tag -->
+		<visual>
+			<!-- How to place and rotate the mesh w.r.t. the xyz axis of its link -->
+			<!-- These values represent the placement and the orientation of the mesh relative to the link it belongs (the xyz axis of the `base_link`) -->
+			<!-- In other words, this `origin` tag is used for visualization and simulation. It is different with the `origin` tag of `joint` -->
+			<!-- `x = y = -0.5` means that we want to place this mesh at the position of x = -0.5 and y = -0.5 w.r.t. the xyz axis of the `base_link`  -->
+			<origin rpy="0 0 0" xyz="-0.5 -0.5 0" />  <!-- `rpy` defines the orientation and `xyz` defines the position -->
+			<geometry>
+				<!-- Mesh file to render -->
 				<mesh filename="package://arduinobot_description/meshes/basement.STL"
 					scale="0.01 0.01 0.01" />
@@ -41,74 +63,152 @@
 		</collision>
 	</link>
+	<link name="base_plate">
+		<xacro:default_inertial mass="0.1" />
+		<visual>
+			<origin rpy="0 0 0" xyz="-0.39 -0.39 -0.56"></origin>
+			<geometry>
+				<mesh filename="package://arduinobot_description/meshes/base_plate.STL"
+					scale="0.01 0.01 0.01"></mesh>
+			</geometry>
+		</visual>
+		<collision>
+			<origin rpy="0 0 0" xyz="-0.39 -0.39 -0.56"></origin>
+			<geometry>
+				<mesh filename="package://arduinobot_description/meshes/base_plate.STL"
+					scale="0.01 0.01 0.01"></mesh>
+			</geometry>
+		</collision>
+	</link>
+	<link name="forward_drive_arm">
+		<xacro:default_inertial mass="0.1" />
+		<visual>
+			<origin rpy="0 -${PI/2} ${PI/2}" xyz="0.19 0.06 -0.08"></origin>
+			<geometry>
+				<mesh filename="package://arduinobot_description/meshes/forward_drive_arm.STL"
+					scale="0.01 0.01 0.01"></mesh>
+			</geometry>
+		</visual>
+		<collision>
+			<origin rpy="0 -${PI/2} ${PI/2}" xyz="0.19 0.06 -0.08"></origin>
+			<geometry>
+				<mesh filename="package://arduinobot_description/meshes/forward_drive_arm.STL"
+					scale="0.01 0.01 0.01"></mesh>
+			</geometry>
+		</collision>
+	</link>
+	<link name="horizontal_arm">
+		<xacro:default_inertial mass="0.1" />
+		<visual>
+			<origin rpy="${PI/2} 0 ${PI/2}" xyz="-0.03 -0.4 -0.06"></origin>
+			<geometry>
+				<mesh filename="package://arduinobot_description/meshes/horizontal_arm.STL"
+					scale="0.01 0.01 0.01"></mesh>
+			</geometry>
+		</visual>
+		<collision>
+			<origin rpy="${PI/2} 0 ${PI/2}" xyz="-0.03 -0.4 -0.06"></origin>
+			<geometry>
+				<mesh filename="package://arduinobot_description/meshes/horizontal_arm.STL"
+					scale="0.01 0.01 0.01"></mesh>
+			</geometry>
+		</collision>
+	</link>
+	<link name="claw_support">
+		<xacro:default_inertial mass="0.05" />
+		<visual>
+			<origin rpy="0 0 ${PI/2}" xyz="0 -0.05 -0.15"></origin>
+			<geometry>
+				<mesh filename="package://arduinobot_description/meshes/claw_support.STL"
+					scale="0.01 0.01 0.01"></mesh>
+			</geometry>
+		</visual>
+		<collision>
+			<origin rpy="0 0 ${PI/2}" xyz="0 -0.05 -0.15"></origin>
+			<geometry>
+				<mesh filename="package://arduinobot_description/meshes/claw_support.STL"
+					scale="0.01 0.01 0.01"></mesh>
+			</geometry>
+		</collision>
+	</link>
+	<link name="gripper_right">
+		<xacro:default_inertial mass="0.01" />
+		<visual>
+			<origin xyz="-0.1 0.5 -0.1" rpy="0 0 -${PI/2}"></origin>
+			<geometry>
+				<mesh filename="package://arduinobot_description/meshes/right_finger.STL"
+					scale="0.01 0.01 0.01"></mesh>
+			</geometry>
+		</visual>
+		<collision>
+			<origin xyz="-0.1 0.5 -0.1" rpy="0 0 -${PI/2}"></origin>
+			<geometry>
+				<mesh filename="package://arduinobot_description/meshes/right_finger.STL"
+					scale="0.01 0.01 0.01"></mesh>
+			</geometry>
+		</collision>
+	</link>
+	<link name="gripper_left">
+		<xacro:default_inertial mass="0.01" />
+		<visual>
+			<origin xyz="-0.04 0.5 -0.1" rpy="0 0 -${PI/2}"></origin>
+			<geometry>
+				<mesh filename="package://arduinobot_description/meshes/left_finger.STL"
+					scale="0.01 0.01 0.01"></mesh>
+			</geometry>
+		</visual>
+		<collision>
+			<origin xyz="-0.04 0.5 -0.1" rpy="0 0 -${PI/2}"></origin>
+			<geometry>
+				<mesh filename="package://arduinobot_description/meshes/left_finger.STL"
+					scale="0.01 0.01 0.01"></mesh>
+			</geometry>
+		</collision>
+	</link>
+	<link name="rgb_camera">
+		<xacro:default_inertial mass="0.001" />
+		<visual>
+			<origin xyz="-0.08 0.125 0.125" rpy="-${PI/2} 0 -${PI/2}"></origin>
+			<geometry>
+				<mesh filename="package://arduinobot_description/meshes/pi_camera.STL"
+					scale="0.01 0.01 0.01"></mesh>
+			</geometry>
+		</visual>
+		<collision>
+			<origin xyz="-0.08 0.125 0.125" rpy="-${PI/2} 0 -${PI/2}"></origin>
+			<geometry>
+				<mesh filename="package://arduinobot_description/meshes/pi_camera.STL"
+					scale="0.01 0.01 0.01"></mesh>
+			</geometry>
+		</collision>
+	</link>
+	<!-- *********** JOINTS *********** -->
+	<!-- `fixed` means the `child` cannot move, rotate or translate w.r.t the `parent` -->
 	<joint name="virtual_joint" type="fixed">
 		<parent link="world" />
 		<child link="base_link" />
+		<!-- How to place and rotate the axis of the `child` link w.r.t. the `parent` link -->
+		<!-- This `origin` tag express the transformation matrix between the `child` and the `world`. The type is `fixed` means that the transformation matrix is zero -->
+		<!-- `rpy = xyz = 0 0 0` means that the `base_link` and `world` have the same center, so the `base_link` is exactly oriented and positioned the same as the world frame (xyz axis of the `base_link` exactly overlap the xyz of the `world`) -->
+		<!-- We can the the `origin` tag express how we place and rotate the XYZ axes of the `child` and `parent` link -->
 		<origin rpy="0 0 0" xyz="0 0 0" />
 	</joint>
-	<link name="base_plate">
-		<xacro:default_inertial mass="0.1" />
-		<visual>
-			<origin rpy="0 0 0" xyz="-0.39 -0.39 -0.56"></origin>
-			<geometry>
-				<mesh filename="package://arduinobot_description/meshes/base_plate.STL"
-					scale="0.01 0.01 0.01"></mesh>
-			</geometry>
-		</visual>
-		<collision>
-			<origin rpy="0 0 0" xyz="-0.39 -0.39 -0.56"></origin>
-			<geometry>
-				<mesh filename="package://arduinobot_description/meshes/base_plate.STL"
-					scale="0.01 0.01 0.01"></mesh>
-			</geometry>
-		</collision>
-	</link>
+	<!-- `revolute` means the `child` can rotate w.r.t. its `parent` (movable joint) -->
 	<joint name="joint_1" type="revolute">
 		<parent link="base_link"></parent>
 		<child link="base_plate"></child>
-		<axis xyz="0 0 1"></axis>
+		<axis xyz="0 0 1"></axis>  <!-- Rotation axis: 0 0 1 means that the `child` rotate around the z axis -->
+		<!-- `rpy` express the rotation and `xyz` express the orientation of the `child` w.r.t. its `parent` -->
+		<!-- the `base_plate` is oriented the same way as the `base_link`, so the `rpy` = 0 0 0. Also, the `base_plate` is translated along the z axis by 3.07cm -->
 		<origin rpy="0 0 0" xyz="0 0 0.307"></origin>
+		<!-- The limit of the rotation ranges from -90 degree to 90 degree  -->
 		<limit lower="-${PI/2}" upper="${PI/2}" effort="${effort}" velocity="${velocity}"></limit>
 	</joint>
-	<link name="forward_drive_arm">
-		<xacro:default_inertial mass="0.1" />
-		<visual>
-			<origin rpy="0 -${PI/2} ${PI/2}" xyz="0.19 0.06 -0.08"></origin>
-			<geometry>
-				<mesh filename="package://arduinobot_description/meshes/forward_drive_arm.STL"
-					scale="0.01 0.01 0.01"></mesh>
-			</geometry>
-		</visual>
-		<collision>
-			<origin rpy="0 -${PI/2} ${PI/2}" xyz="0.19 0.06 -0.08"></origin>
-			<geometry>
-				<mesh filename="package://arduinobot_description/meshes/forward_drive_arm.STL"
-					scale="0.01 0.01 0.01"></mesh>
-			</geometry>
-		</collision>
-	</link>
 	<joint name="joint_2" type="revolute">
 		<parent link="base_plate"></parent>
 		<child link="forward_drive_arm"></child>
 		<axis xyz="1 0 0"></axis>
-		<origin rpy="0 0 0" xyz="-0.02 0 0.35"></origin>
+		<origin rpy="0 0 0" xyz="0.02 0 0.35"></origin>
 		<limit lower="-${PI/2}" upper="${PI/2}" effort="${effort}" velocity="${velocity}"></limit>
 	</joint>
-	<link name="horizontal_arm">
-		<xacro:default_inertial mass="0.1" />
-		<visual>
-			<origin rpy="${PI/2} 0 ${PI/2}" xyz="-0.03 -0.4 -0.06"></origin>
-			<geometry>
-				<mesh filename="package://arduinobot_description/meshes/horizontal_arm.STL"
-					scale="0.01 0.01 0.01"></mesh>
-			</geometry>
-		</visual>
-		<collision>
-			<origin rpy="${PI/2} 0 ${PI/2}" xyz="-0.03 -0.4 -0.06"></origin>
-			<geometry>
-				<mesh filename="package://arduinobot_description/meshes/horizontal_arm.STL"
-					scale="0.01 0.01 0.01"></mesh>
-			</geometry>
-		</collision>
-	</link>
 	<joint name="joint_3" type="revolute">
 		<parent link="forward_drive_arm"></parent>
@@ -118,21 +218,4 @@
 		<limit lower="-${PI/2}" upper="${PI/2}" effort="${effort}" velocity="${velocity}"></limit>
 	</joint>
-	<link name="claw_support">
-		<xacro:default_inertial mass="0.05" />
-		<visual>
-			<origin rpy="0 0 ${PI/2}" xyz="0 -0.05 -0.15"></origin>
-			<geometry>
-				<mesh filename="package://arduinobot_description/meshes/claw_support.STL"
-					scale="0.01 0.01 0.01"></mesh>
-			</geometry>
-		</visual>
-		<collision>
-			<origin rpy="0 0 ${PI/2}" xyz="0 -0.05 -0.15"></origin>
-			<geometry>
-				<mesh filename="package://arduinobot_description/meshes/claw_support.STL"
-					scale="0.01 0.01 0.01"></mesh>
-			</geometry>
-		</collision>
-	</link>
 	<joint name="horizontal_arm_to_claw_support" type="fixed">
 		<parent link="horizontal_arm"></parent>
@@ -140,38 +223,4 @@
 		<origin xyz="0 0.82 0" rpy="0 0 0"></origin>
 	</joint>
-	<link name="gripper_right">
-		<xacro:default_inertial mass="0.01" />
-		<visual>
-			<origin xyz="-0.1 0.5 -0.1" rpy="0 0 -${PI/2}"></origin>
-			<geometry>
-				<mesh filename="package://arduinobot_description/meshes/right_finger.STL"
-					scale="0.01 0.01 0.01"></mesh>
-			</geometry>
-		</visual>
-		<collision>
-			<origin xyz="-0.1 0.5 -0.1" rpy="0 0 -${PI/2}"></origin>
-			<geometry>
-				<mesh filename="package://arduinobot_description/meshes/right_finger.STL"
-					scale="0.01 0.01 0.01"></mesh>
-			</geometry>
-		</collision>
-	</link>
-	<link name="gripper_left">
-		<xacro:default_inertial mass="0.01" />
-		<visual>
-			<origin xyz="-0.04 0.5 -0.1" rpy="0 0 -${PI/2}"></origin>
-			<geometry>
-				<mesh filename="package://arduinobot_description/meshes/left_finger.STL"
-					scale="0.01 0.01 0.01"></mesh>
-			</geometry>
-		</visual>
-		<collision>
-			<origin xyz="-0.04 0.5 -0.1" rpy="0 0 -${PI/2}"></origin>
-			<geometry>
-				<mesh filename="package://arduinobot_description/meshes/left_finger.STL"
-					scale="0.01 0.01 0.01"></mesh>
-			</geometry>
-		</collision>
-	</link>
 	<joint name="joint_4" type="revolute">
 		<parent link="claw_support"></parent>
@@ -186,24 +235,14 @@
 		<axis xyz="0 0 1"></axis>
 		<origin rpy="0 0 0" xyz="-0.22 0.13 -0.1"></origin>
+		<!--
+			Since the gripper left and right will move together, they are composed of a gear
+			system that ensures that they open and close together so that they open and
+			close by the same angle => We should use `mimic` tag to perform this action.
+			multiplier="-1" indicates that gripper left and right rotate in an opposite
+			direction
+		-->
 		<mimic joint="joint_4" multiplier="-1"></mimic>
 		<limit lower="0.0" upper="${PI/2}" effort="${effort}" velocity="${velocity}"></limit>
 	</joint>
-	<link name="rgb_camera">
-		<xacro:default_inertial mass="0.001" />
-		<visual>
-			<origin xyz="-0.08 0.125 0.125" rpy="-${PI/2} 0 -${PI/2}"></origin>
-			<geometry>
-				<mesh filename="package://arduinobot_description/meshes/pi_camera.STL"
-					scale="0.01 0.01 0.01"></mesh>
-			</geometry>
-		</visual>
-		<collision>
-			<origin xyz="-0.08 0.125 0.125" rpy="-${PI/2} 0 -${PI/2}"></origin>
-			<geometry>
-				<mesh filename="package://arduinobot_description/meshes/pi_camera.STL"
-					scale="0.01 0.01 0.01"></mesh>
-			</geometry>
-		</collision>
-	</link>
 	<joint name="joint_6" type="fixed">
 		<parent link="base_link" />
@@ -216,2 +255,3 @@
 	<xacro:default_transmission number="4"/>
 </robot>
+<!-- We need to INSTALL this `urdf` folder and `meshes` folder so that these folders are recognized within our package -->
