Commit message: add all script in Sec. 9

File: src/arduinobot_description/urdf/arduinobot.urdf.xacro (robot description, xacro)
@@ -2,4 +2,5 @@
 <!-- We are using the xacro format, not plain urdf => we need to indicate where the definition of this format is located  -->
 <robot xmlns:xacro="http://www.ros.org/wiki/xacro" name="arduinobot">
+	<xacro:arg name="is_sim" default="true" />
 	<!-- Include within this model the new file that we have created. -->
 	<xacro:include filename="$(find arduinobot_description)/urdf/arduinobot_gazebo.xacro" />

File: src/arduinobot_description/urdf/arduinobot_ros2_control.xacro (robot description, xacro)
@@ -1,5 +1,4 @@
 <?xml version="1.0"?>
 <robot xmlns:xacro="http://www.ros.org/wiki/xacro" name="arduinobot">
-	<xacro:property name="PI" value="3.14159" />
     <!--
         ros2_control tag used to config and interface the robot's
@@ -7,23 +6,48 @@
     -->
     <ros2_control name="RobotSystem" type="system">
-        <!--
-            Indicate the type of hardware that makes up the system
-            and that we want to interface with the ROS2 control
-            library.
-        -->
-        <hardware>
+	    <xacro:property name="PI" value="3.14159" />
+        <xacro:if value="$(arg is_sim)">
             <!--
-                Since we only have the simulated version of the
-                robot in Gazebo, the hardware is represented by
-                the gazebo itself. So we use the plugin that is
-                GazeboSystem.
-                This component needs to be changed when we will
-                create our real robot, and so when we are going
-                to need to interface the control system with
-                the actual hardware. So with the real motors
-                instead of with the gazebo control library.
+                Indicate the type of hardware that makes up the system
+                and that we want to interface with the ROS2 control
+                library.
             -->
-            <plugin>gazebo_ros2_control/GazeboSystem</plugin>
-        </hardware>
+            <hardware>
+                <!--
+                    Since we only have the simulated version of the
+                    robot in Gazebo, the hardware is represented by
+                    the gazebo itself. So we use the plugin that is
+                    GazeboSystem.
+                    This component needs to be changed when we will
+                    create our real robot, and so when we are going
+                    to need to interface the control system with
+                    the actual hardware. So with the real motors
+                    instead of with the gazebo control library.
+                -->
+                <plugin>gazebo_ros2_control/GazeboSystem</plugin>
+            </hardware>
+            <joint name="joint_5">
+                <!--
+                    To let the control system and also to inform the
+                    ROS2  control library of the relationship of
+                    joint_4 and joint_5, we need to set two
+                    parameters that are mimic and multiplier.
+                -->
+                <param name="mimic">joint_4</param>
+                <param name="multiplier">-1</param>
+                <command_interface name="position">
+                    <param name="min">0.0</param>
+                    <param name="max">${PI/2}</param>
+                </command_interface>
+                <state_interface name="position">
+                </state_interface>
+            </joint>
+        </xacro:if>
+        <xacro_unless value="$(arg is_sim)">
+            <hardware>
+                <plugin>arduinobot_controller/ArduinobotInterface</plugin>
+                <param name="port">/dev/ttyACM0</param>
+            </hardware>
+        </xacro_unless>
         <!--
             Now we need to define also the interface that each
@@ -88,20 +112,4 @@
             </state_interface>
         </joint>
-        <joint name="joint_5">
-            <!--
-                To let the control system and also to inform the
-                ROS2  control library of the relationship of
-                joint_4 and joint_5, we need to set two
-                parameters that are mimic and multiplier.
-            -->
-            <param name="mimic">joint_4</param>
-            <param name="multiplier">-1</param>
-            <command_interface name="position">
-                <param name="min">0.0</param>
-                <param name="max">${PI/2}</param>
-            </command_interface>
-            <state_interface name="position">
-            </state_interface>
-        </joint>
     </ros2_control>
 </robot>
